Commit message: copter not flying

File: Tools/rotors_description/urdf/iris_base.xacro (robot description, xacro)
@@ -52,5 +52,5 @@
   </xacro:if>
   <!-- Instantiate a controller. -->
-  <xacro:controller_plugin_macro namespace="${namespace}" imu_sub_topic="imu" />
+  <!-- <xacro:controller_plugin_macro namespace="${namespace}" imu_sub_topic="imu" /> -->
   <!-- Mount an ADIS16448 IMU. -->
   <!-- <xacro:default_imu namespace="${namespace}" parent_link="${namespace}/base_link" /> -->

File: Tools/rotors_description/urdf/mav_vi_name.urdf (robot description, URDF)
Before this commit: robot iris, 16 links, 15 joints
Links:
- removed link iris/base_link
- removed link iris/base_link_inertia
- removed link iris/imu_link
- removed link iris/odometry_sensor1_link
- removed link iris/rotor_0
- removed link iris/rotor_1
- removed link iris/rotor_2
- removed link iris/rotor_3
- removed link iris/vi_sensor/camera_depth_link
- removed link iris/vi_sensor/camera_depth_optical_center_link
- removed link iris/vi_sensor/camera_left_link
- removed link iris/vi_sensor/camera_left_optical_link
- removed link iris/vi_sensor/camera_right_link
- removed link iris/vi_sensor/ground_truth/odometry_sensor_link
- removed link iris/vi_sensor/imu_link
- removed link iris/vi_sensor/vi_sensor_link
- added link /base_link
- added link /base_link_inertia, mass 1.5; collision box size=0.47 0.47 0.11; visual mesh filename=package://rotors_description/meshes/iris.dae scale=1 1 1
- added link /imu_link, mass 0.015
- added link /odometry_sensor1_link, mass 1e-05
- added link /rotor_0, mass 0.005; collision cylinder length=0.005 radius=0.1; visual mesh filename=package://rotors_description/meshes/propeller_ccw.dae scale=0.1 0.1 0.1
- added link /rotor_1, mass 0.005; collision cylinder length=0.005 radius=0.1; visual mesh filename=package://rotors_description/meshes/propeller_ccw.dae scale=0.1 0.1 0.1
- added link /rotor_2, mass 0.005; collision cylinder length=0.005 radius=0.1; visual mesh filename=package://rotors_description/meshes/propeller_cw.dae scale=0.1 0.1 0.1
- added link /rotor_3, mass 0.005; collision cylinder length=0.005 radius=0.1; visual mesh filename=package://rotors_description/meshes/propeller_cw.dae scale=0.1 0.1 0.1
- added link /vi_sensor/camera_depth_link, mass 1e-5; collision cylinder length=0.01 radius=0.007
- added link /vi_sensor/camera_depth_optical_center_link
- added link /vi_sensor/camera_left_link, mass 1e-5; collision cylinder length=0.01 radius=0.007
- added link /vi_sensor/camera_left_optical_link
- added link /vi_sensor/camera_right_link, mass 1e-5; collision cylinder length=0.01 radius=0.007
- added link /vi_sensor/ground_truth/odometry_sensor_link, mass 1e-05
- added link /vi_sensor/imu_link, mass 0.015
- added link /vi_sensor/vi_sensor_link, mass 0.13; collision box size=0.03 0.133 0.057; visual mesh filename=package://rotors_description/meshes/vi_sensor.dae scale=1 1 1
Joints:
- removed joint iris/base_joint
- removed joint iris/imu_joint
- removed joint iris/odometry_sensor1_joint
- removed joint iris/rotor_0_joint
- removed joint iris/rotor_1_joint
- removed joint iris/rotor_2_joint
- removed joint iris/rotor_3_joint
- removed joint iris/vi_sensor/camera_depth_joint
- removed joint iris/vi_sensor/camera_depth_optical_center_joint
- removed joint iris/vi_sensor/camera_left_joint
- removed joint iris/vi_sensor/camera_left_optical_joint
- removed joint iris/vi_sensor/camera_right_joint
- removed joint iris/vi_sensor/ground_truth/odometry_sensor_joint
- removed joint iris/vi_sensor/imu_joint
- removed joint iris/vi_sensor_vi_sensor_joint
- added joint /base_joint: type fixed, parent /base_link, child /base_link_inertia, origin xyz=0 0 0 rpy=0 0 0
- added joint /imu_joint: type revolute, parent /base_link, child /imu_link, origin xyz=0 0 0 rpy=0 0 0, limit lower=0 upper=0 effort=0 velocity=0
- added joint /odometry_sensor1_joint: type revolute, parent /base_link, child /odometry_sensor1_link, origin xyz=0.0 0.0 0.0 rpy=0.0 0.0 0.0, limit lower=0 upper=0 effort=0 velocity=0
- added joint /rotor_0_joint: type continuous, parent /base_link, child /rotor_0, origin xyz=0.13 -0.22 0.023 rpy=0 0 0, axis 0 0 1
- added joint /rotor_1_joint: type continuous, parent /base_link, child /rotor_1, origin xyz=-0.13 0.2 0.023 rpy=0 0 0, axis 0 0 1
- added joint /rotor_2_joint: type continuous, parent /base_link, child /rotor_2, origin xyz=0.13 0.22 0.023 rpy=0 0 0, axis 0 0 1
- added joint /rotor_3_joint: type continuous, parent /base_link, child /rotor_3, origin xyz=-0.13 -0.2 0.023 rpy=0 0 0, axis 0 0 1
- added joint /vi_sensor/camera_depth_joint: type fixed, parent /vi_sensor/vi_sensor_link, child /vi_sensor/camera_depth_link, origin xyz=0.015 0.055 0.0065 rpy=0 0 0, limit lower=0 upper=0 effort=0 velocity=0
- added joint /vi_sensor/camera_depth_optical_center_joint: type fixed, parent /vi_sensor/camera_depth_link, child /vi_sensor/camera_depth_optical_center_link, origin xyz=0 0 0 rpy=-1.5707963268 0 -1.5707963268, limit lower=0 upper=0 effort=0 velocity=0
- added joint /vi_sensor/camera_left_joint: type fixed, parent /vi_sensor/vi_sensor_link, child /vi_sensor/camera_left_link, origin xyz=0.015 0.055 0.0065 rpy=0 0 0
- added joint /vi_sensor/camera_left_optical_joint: type fixed, parent /vi_sensor/camera_left_link, child /vi_sensor/camera_left_optical_link, origin xyz=0 0 0 rpy=-1.5707963268 0 -1.5707963268
- added joint /vi_sensor/camera_right_joint: type fixed, parent /vi_sensor/vi_sensor_link, child /vi_sensor/camera_right_link, origin xyz=0.015 -0.055 0.0065 rpy=0 0 0
- added joint /vi_sensor/ground_truth/odometry_sensor_joint: type revolute, parent /vi_sensor/vi_sensor_link, child /vi_sensor/ground_truth/odometry_sensor_link, origin xyz=0.0 0.0 0.0 rpy=0.0 0.0 0.0, limit lower=0 upper=0 effort=0 velocity=0
- added joint /vi_sensor/imu_joint: type revolute, parent /vi_sensor/vi_sensor_link, child /vi_sensor/imu_link, origin xyz=0.015 0 0.0113 rpy=0 0 0, limit lower=0 upper=0 effort=0 velocity=0
- added joint /vi_sensor_vi_sensor_joint: type fixed, parent /base_link, child /vi_sensor/vi_sensor_link, origin xyz=0.1 0.0 -0.03 rpy=0.0 0.1 0.0

Commit message: not working yet

File: Tools/rotors_description/urdf/iris_base.xacro (robot description, xacro)
@@ -74,13 +74,13 @@
   <origin xyz="0 0 0" rpy="0 0 0" />
 </xacro:imu_plugin_macro>
+<xacro:ground_truth_imu_and_odometry namespace="${namespace}" parent_link="${namespace}/base_link" />
   <xacro:if value="$(arg enable_ground_truth)">
-    <xacro:ground_truth_imu_and_odometry namespace="${namespace}" parent_link="${namespace}/base_link" />
-  </xacro:if>
-  <!-- <xacro:if value="$(arg enable_ground_truth)"> -->
-    <!-- Mount an IMU providing ground truth. -->
-    <!-- <xacro:imu_plugin_macro
+</xacro:if>
+  <!-- <xacro:if value="$(arg enable_ground_truth)">
+    Mount an IMU providing ground truth.
+    <xacro:imu_plugin_macro
       namespace="${namespace}"
       imu_suffix="gt"
-      parent_link="${namespace}/base_link"
+      parent_link="${parent_link}"
       imu_topic="ground_truth/imu"
       mass_imu_sensor="0.00001"
@@ -92,19 +92,18 @@
       accelerometer_random_walk="0.0"
       accelerometer_bias_correlation_time="300.0"
-      accelerometer_turn_on_bias_sigma="0.0"
-    >
+      accelerometer_turn_on_bias_sigma="0.0">
       <inertia ixx="0.00001" ixy="0.0" ixz="0.0" iyy="0.00001" iyz="0.0" izz="0.00001" />
       <origin xyz="0 0 0" rpy="0 0 0" />
-    </xacro:imu_plugin_macro> -->
-    <!-- Mount a generic odometry sensor providing ground truth. -->
-    <!-- <xacro:odometry_plugin_macro
-      namespace="${namespace}/ground_truth"
+    </xacro:imu_plugin_macro>
+    Mount a generic odometry sensor providing ground truth.
+    <xacro:odometry_plugin_macro
+      namespace="${namespace}"
       odometry_sensor_suffix="gt"
-      parent_link="base_link"
-      pose_topic="pose"
-      pose_with_covariance_topic="pose_with_covariance"
-      position_topic="position"
-      transform_topic="transform"
-      odometry_topic="odometry"
+      parent_link="${parent_link}"
+      pose_topic="ground_truth/pose"
+      pose_with_covariance_topic="ground_truth/pose_with_covariance"
+      position_topic="ground_truth/position"
+      transform_topic="ground_truth/transform"
+      odometry_topic="ground_truth/odometry"
       parent_frame_id="world"
       child_frame_id="${namespace}/base_link"
@@ -123,9 +122,8 @@
       enable_odometry_map="false"
       odometry_map=""
-      image_scale=""
-    >
-      <inertia ixx="0.00001" ixy="0.0" ixz="0.0" iyy="0.00001" iyz="0.0" izz="0.00001" />  -->
-      <!-- [kg.m^2] [kg.m^2] [kg.m^2] [kg.m^2] [kg.m^2] [kg.m^2] -->
-      <!-- <origin xyz="0.0 0.0 0.0" rpy="0.0 0.0 0.0" />
+      image_scale="">
+      <inertia ixx="0.00001" ixy="0.0" ixz="0.0" iyy="0.00001" iyz="0.0" izz="0.00001" />
+      [kg.m^2] [kg.m^2] [kg.m^2] [kg.m^2] [kg.m^2] [kg.m^2]
+       <origin xyz="0.0 0.0 0.0" rpy="0.0 0.0 0.0" />
     </xacro:odometry_plugin_macro>
   </xacro:if> -->

File: Tools/rotors_description/urdf/iris_base_sitl.xacro (robot description, xacro)
@@ -79,7 +79,7 @@
     accelerometer_turn_on_bias_sigma="0.1960"
   >
-    <inertia ixx="0.00001" ixy="0.0" ixz="0.0" iyy="0.00001" iyz="0.0" izz="0.00001" />
-    <origin xyz="0 0 0" rpy="0 0 0" />
-  </xacro:imu_plugin_macro>
+  <inertia ixx="0.00001" ixy="0.0" ixz="0.0" iyy="0.00001" iyz="0.0" izz="0.00001" />
+  <origin xyz="0 0 0" rpy="0 0 0" />
+</xacro:imu_plugin_macro>
   <xacro:if value="$(arg enable_ground_truth)">
     <!-- Mount an IMU providing ground truth. -->
